Commit message: Initial tuning of control board gains

File: retargeting-models/robots/nao/model.urdf (robot description, URDF)
Before this commit: robot NaoH25V40, 83 links, 82 joints
Links:
- removed link LFinger11_link
- removed link LFinger12_link
- removed link LFinger13_link
- removed link LFinger21_link
- removed link LFinger22_link
- removed link LFinger23_link
- removed link LThumb1_link
- removed link LThumb2_link
- removed link RFinger11_link
- removed link RFinger12_link
- removed link RFinger13_link
- removed link RFinger21_link
- removed link RFinger22_link
- removed link RFinger23_link
- removed link RThumb1_link
- removed link RThumb2_link
Joints:
- removed joint LFinger11
- removed joint LFinger12
- removed joint LFinger13
- removed joint LFinger21
- removed joint LFinger22
- removed joint LFinger23
- removed joint LThumb1
- removed joint LThumb2
- removed joint RFinger11
- removed joint RFinger12
- removed joint RFinger13
- removed joint RFinger21
- removed joint RFinger22
- removed joint RFinger23
- removed joint RThumb1
- removed joint RThumb2

Commit message: Final tuning of nao control boards and add world to based fixed joint

File: retargeting-models/robots/nao/model.urdf (robot description, URDF)
Before this commit: robot NaoH25V40, 67 links, 66 joints
Links:
- added link world
Joints:
- added joint world_base_fixed_joint: type fixed, parent world, child base_link, origin xyz=0 0 1 rpy=0 -0 0, axis 0 0 0
