Commit message: Rearrange directory structure

File: robots/baxter/model.urdf (robot description, URDF)
Before this commit: robot baxter, 50 links, 49 joints
Links:
- link head: geometry collision sphere radius=0.001; visual mesh filename=package://retargeting-robot-models/robots/baxter/meshes/hea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
- link left_lower_elbow: geometry collision cylinder length=0.10 radius=0.06; visual mesh filename=package://retargeting-robot-models/robots/baxter/meshes/low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
- link left_lower_forearm: geometry collision cylinder length=0.10 radius=0.06; visual mesh filename=package://retargeting-robot-models/robots/baxter/meshes/low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
- link left_lower_shoulder: geometry collision cylinder length=0.12 radius=0.06; visual mesh filename=package://retargeting-robot-models/robots/baxter/meshes/low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
- link left_upper_elbow: geometry collision cylinder length=0.107 radius=0.06; visual mesh filename=package://retargeting-robot-models/robots/baxter/meshes/upp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
- link left_upper_forearm: geometry collision cylinder length=0.088 radius=0.06; visual mesh filename=package://retargeting-robot-models/robots/baxter/meshes/upp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
- link left_upper_shoulder: geometry collision cylinder length=0.2722 radius=0.06; visual mesh filename=package://retargeting-robot-models/robots/baxter/meshes/upp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
- link left_wrist: geometry collision cylinder length=0.165 radius=0.06; visual mesh filename=package://retargeting-robot-models/robots/baxter/meshes/wri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
- link pedestal: geometry collision mesh filename=package://retargeting-robot-models/robots/baxter/meshes/bas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; visual mesh filename=package://retargeting-robot-models/robots/baxter/meshes/bas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
- link right_lower_elbow: geometry collision cylinder length=0.10 radius=0.06; visual mesh filename=package://retargeting-robot-models/robots/baxter/meshes/low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
- link right_lower_forearm: geometry collision cylinder length=0.10 radius=0.06; visual mesh filename=package://retargeting-robot-models/robots/baxter/meshes/low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
- link right_lower_shoulder: geometry collision cylinder length=0.12 radius=0.06; visual mesh filename=package://retargeting-robot-models/robots/baxter/meshes/low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
- link right_upper_elbow: geometry collision cylinder length=0.107 radius=0.06; visual mesh filename=package://retargeting-robot-models/robots/baxter/meshes/upp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
- link right_upper_forearm: geometry collision cylinder length=0.088 radius=0.06; visual mesh filename=package://retargeting-robot-models/robots/baxter/meshes/upp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
- link right_upper_shoulder: geometry collision cylinder length=0.2722 radius=0.06; visual mesh filename=package://retargeting-robot-models/robots/baxter/meshes/upp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
- link right_wrist: geometry collision cylinder length=0.165 radius=0.06; visual mesh filename=package://retargeting-robot-models/robots/baxter/meshes/wri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
- link screen: geometry collision sphere radius=0.001; visual mesh filename=package://retargeting-robot-models/robots/baxter/meshes/hea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
- link torso: geometry collision mesh filename=package://retargeting-robot-models/robots/baxter/meshes/tor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; visual mesh filename=package://retargeting-robot-models/robots/baxter/meshes/tor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

File: robots/nao/model.urdf (robot description, URDF)
Before this commit: robot NaoH25V40, 68 links, 67 joints
Links:
- link Head: geometry collision mesh filename=package://retargeting-robot-models/robots/nao/nao_meshes/me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 scale=0.1 0.1 0.1; visual mesh filename=package://retargeting-robot-models/robots/nao/nao_meshes/me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 scale=0.1 0.1 0.1
- link LAnklePitch: geometry collision mesh filename=package://retargeting-robot-models/robots/nao/nao_meshes/me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 scale=0.1 0.1 0.1; visual mesh filename=package://retargeting-robot-models/robots/nao/nao_meshes/me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 scale=0.1 0.1 0.1
- link LBicep: geometry collision mesh filename=package://retargeting-robot-models/robots/nao/nao_meshes/me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 scale=0.1 0.1 0.1; visual mesh filename=package://retargeting-robot-models/robots/nao/nao_meshes/me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 scale=0.1 0.1 0.1
- link LForeArm: geometry collision mesh filename=package://retargeting-robot-models/robots/nao/nao_meshes/me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 scale=0.1 0.1 0.1; visual mesh filename=package://retargeting-robot-models/robots/nao/nao_meshes/me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 scale=0.1 0.1 0.1
- link LHip: geometry collision mesh filename=package://retargeting-robot-models/robots/nao/nao_meshes/me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 scale=0.1 0.1 0.1; visual mesh filename=package://retargeting-robot-models/robots/nao/nao_meshes/me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 scale=0.1 0.1 0.1
- link LPelvis: geometry collision mesh filename=package://retargeting-robot-models/robots/nao/nao_meshes/me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 scale=0.1 0.1 0.1; visual mesh filename=package://retargeting-robot-models/robots/nao/nao_meshes/me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 scale=0.1 0.1 0.1
- link LShoulder: geometry collision mesh filename=package://retargeting-robot-models/robots/nao/nao_meshes/me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 scale=0.1 0.1 0.1; visual mesh filename=package://retargeting-robot-models/robots/nao/nao_meshes/me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 scale=0.1 0.1 0.1
- link LThigh: geometry collision mesh filename=package://retargeting-robot-models/robots/nao/nao_meshes/me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 scale=0.1 0.1 0.1; visual mesh filename=package://retargeting-robot-models/robots/nao/nao_meshes/me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 scale=0.1 0.1 0.1
- link LTibia: geometry collision mesh filename=package://retargeting-robot-models/robots/nao/nao_meshes/me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 scale=0.1 0.1 0.1; visual mesh filename=package://retargeting-robot-models/robots/nao/nao_meshes/me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 scale=0.1 0.1 0.1
- link Neck: geometry collision mesh filename=package://retargeting-robot-models/robots/nao/nao_meshes/me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 scale=0.1 0.1 0.1; visual mesh filename=package://retargeting-robot-models/robots/nao/nao_meshes/me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 scale=0.1 0.1 0.1
- link RAnklePitch: geometry collision mesh filename=package://retargeting-robot-models/robots/nao/nao_meshes/me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 scale=0.1 0.1 0.1; visual mesh filename=package://retargeting-robot-models/robots/nao/nao_meshes/me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 scale=0.1 0.1 0.1
- link RBicep: geometry collision mesh filename=package://retargeting-robot-models/robots/nao/nao_meshes/me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 scale=0.1 0.1 0.1; visual mesh filename=package://retargeting-robot-models/robots/nao/nao_meshes/me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 scale=0.1 0.1 0.1
- link RForeArm: geometry collision mesh filename=package://retargeting-robot-models/robots/nao/nao_meshes/me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 scale=0.1 0.1 0.1; visual mesh filename=package://retargeting-robot-models/robots/nao/nao_meshes/me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 scale=0.1 0.1 0.1
- link RHip: geometry collision mesh filename=package://retargeting-robot-models/robots/nao/nao_meshes/me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 scale=0.1 0.1 0.1; visual mesh filename=package://retargeting-robot-models/robots/nao/nao_meshes/me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 scale=0.1 0.1 0.1
- link RPelvis: geometry collision mesh filename=package://retargeting-robot-models/robots/nao/nao_meshes/me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 scale=0.1 0.1 0.1; visual mesh filename=package://retargeting-robot-models/robots/nao/nao_meshes/me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 scale=0.1 0.1 0.1
- link RShoulder: geometry collision mesh filename=package://retargeting-robot-models/robots/nao/nao_meshes/me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 scale=0.1 0.1 0.1; visual mesh filename=package://retargeting-robot-models/robots/nao/nao_meshes/me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 scale=0.1 0.1 0.1
- link RThigh: geometry collision mesh filename=package://retargeting-robot-models/robots/nao/nao_meshes/me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 scale=0.1 0.1 0.1; visual mesh filename=package://retargeting-robot-models/robots/nao/nao_meshes/me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 scale=0.1 0.1 0.1
- link RTibia: geometry collision mesh filename=package://retargeting-robot-models/robots/nao/nao_meshes/me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 scale=0.1 0.1 0.1; visual mesh filename=package://retargeting-robot-models/robots/nao/nao_meshes/me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 scale=0.1 0.1 0.1
- link l_ankle: geometry collision mesh filename=package://retargeting-robot-models/robots/nao/nao_meshes/me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 scale=0.1 0.1 0.1; visual mesh filename=package://retargeting-robot-models/robots/nao/nao_meshes/me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 scale=0.1 0.1 0.1
- link l_wrist: geometry collision mesh filename=package://retargeting-robot-models/robots/nao/nao_meshes/me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 scale=0.1 0.1 0.1; visual mesh filename=package://retargeting-robot-models/robots/nao/nao_meshes/me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 scale=0.1 0.1 0.1
- link r_ankle: geometry collision mesh filename=package://retargeting-robot-models/robots/nao/nao_meshes/me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 scale=0.1 0.1 0.1; visual mesh filename=package://retargeting-robot-models/robots/nao/nao_meshes/me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 scale=0.1 0.1 0.1
- link r_wrist: geometry collision mesh filename=package://retargeting-robot-models/robots/nao/nao_meshes/me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 scale=0.1 0.1 0.1; visual mesh filename=package://retargeting-robot-models/robots/nao/nao_meshes/me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 scale=0.1 0.1 0.1
- link torso: geometry collision mesh filename=package://retargeting-robot-models/robots/nao/nao_meshes/me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 scale=0.1 0.1 0.1; visual mesh filename=package://retargeting-robot-models/robots/nao/nao_meshes/me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 scale=0.1 0.1 0.1

Commit message: fake links added for teleoperation

File: robots/baxter/model.urdf (robot description, URDF)
Before this commit: robot baxter, 50 links, 49 joints
Links:
- added link left_lower_elbow_fake, mass 0.0001
- added link left_lower_forearm_fake, mass 0.0001
- added link left_lower_shoulder_fake, mass 0.0001
- added link left_upper_elbow_fake, mass 0.0001
- added link left_upper_forearm_fake, mass 0.0001
- added link left_upper_shoulder_fake, mass 0.0001
- added link left_wrist_fake, mass 0.0001
- added link right_lower_elbow_fake, mass 0.0001
- added link right_lower_forearm_fake, mass 0.0001
- added link right_lower_shoulder_fake, mass 0.0001
- added link right_upper_elbow_fake, mass 0.0001
- added link right_upper_forearm_fake, mass 0.0001
- added link right_upper_shoulder_fake, mass 0.0001
- added link right_wrist_fake, mass 0.0001
Joints:
- added joint j_left_lower_elbow_fake: type fixed, parent left_lower_elbow, child left_lower_elbow_fake, origin xyz=0 0 0 rpy=3.14159265358979 0 1.57079632679, axis 0 0 0
- added joint j_left_lower_forearm_fake: type fixed, parent left_lower_forearm, child left_lower_forearm_fake, origin xyz=0 0 0 rpy=3.14159265358979 0 1.57079632679, axis 0 0 0
- added joint j_left_lower_shoulder_fake: type fixed, parent left_lower_shoulder, child left_lower_shoulder_fake, origin xyz=0 0 0 rpy=1.57079632679 1.57079632679 0, axis 0 0 0
- added joint j_left_upper_elbow_fake: type fixed, parent left_upper_elbow, child left_upper_elbow_fake, origin xyz=0 0 0 rpy=1.57079632679 0 0, axis 0 0 0
- added joint j_left_upper_forearm_fake: type fixed, parent left_upper_forearm, child left_upper_forearm_fake, origin xyz=0 0 0 rpy=1.57079632679 0 0, axis 0 0 0
- added joint j_left_upper_shoulder_fake: type fixed, parent left_upper_shoulder, child left_upper_shoulder_fake, origin xyz=0 0 0 rpy=0 0 -1.57079632679, axis 0 0 0
- added joint j_left_wrist_fake: type fixed, parent left_wrist, child left_wrist_fake, origin xyz=0 0 0 rpy=1.57079632679 0 0, axis 0 0 0
- added joint j_right_lower_elbow_fake: type fixed, parent right_lower_elbow, child right_lower_elbow_fake, origin xyz=0 0 0 rpy=0 0 1.57079632679, axis 0 0 0
- added joint j_right_lower_forearm_fake: type fixed, parent right_lower_forearm, child right_lower_forearm_fake, origin xyz=0 0 0 rpy=0 0 1.57079632679, axis 0 0 0
- added joint j_right_lower_shoulder_fake: type fixed, parent right_lower_shoulder, child right_lower_shoulder_fake, origin xyz=0 0 0 rpy=1.57079632679 -1.57079632679 0, axis 0 0 0
- added joint j_right_upper_elbow_fake: type fixed, parent right_upper_elbow, child right_upper_elbow_fake, origin xyz=0 0 0 rpy=-1.57079632679 0 0, axis 0 0 0
- added joint j_right_upper_forearm_fake: type fixed, parent right_upper_forearm, child right_upper_forearm_fake, origin xyz=0 0 0 rpy=-1.57079632679 0 0, axis 0 0 0
- added joint j_right_upper_shoulder_fake: type fixed, parent right_upper_shoulder, child right_upper_shoulder_fake, origin xyz=0 0 0 rpy=0 0 1.57079632679, axis 0 0 0
- added joint j_right_wrist_fake: type fixed, parent right_wrist, child right_wrist_fake, origin xyz=0 0 0 rpy=-1.57079632679 0 0, axis 0 0 0

File: robots/nao/model.urdf (robot description, URDF)
Before this commit: robot NaoH25V40, 68 links, 67 joints
Links:
- added link LBicep_fake, mass 0.0001
- added link LElbow_fake, mass 0.0001
- added link LForeArm_fake, mass 0.0001
- added link RBicep_fake, mass 0.0001
- added link RElbow_fake, mass 0.0001
- added link RForeArm_fake, mass 0.0001
- added link l_wrist_fake, mass 0.0001
- added link r_wrist_fake, mass 0.0001
Joints:
- added joint j_LBicep_fake: type fixed, parent LBicep, child LBicep_fake, origin xyz=0 0 0 rpy=0 0 -1.57079632679, axis 0 0 0
- added joint j_LElbow_fake: type fixed, parent LElbow, child LElbow_fake, origin xyz=0 0 0 rpy=0 0 -1.57079632679, axis 0 0 0
- added joint j_LForeArm_fake: type fixed, parent LForeArm, child LForeArm_fake, origin xyz=0 0 0 rpy=0 0 -1.57079632679, axis 0 0 0
- added joint j_RBicep_fake: type fixed, parent RBicep, child RBicep_fake, origin xyz=0 0 0 rpy=0 0 1.57079632679, axis 0 0 0
- added joint j_RElbow_fake: type fixed, parent RElbow, child RElbow_fake, origin xyz=0 0 0 rpy=0 0 1.57079632679, axis 0 0 0
- added joint j_RForeArm_fake: type fixed, parent RForeArm, child RForeArm_fake, origin xyz=0 0 0 rpy=0 0 1.57079632679, axis 0 0 0
- added joint j_l_wrist_fake: type fixed, parent l_wrist, child l_wrist_fake, origin xyz=0 0 0 rpy=0 0 -1.57079632679, axis 0 0 0
- added joint j_r_wrist_fake: type fixed, parent r_wrist, child r_wrist_fake, origin xyz=0 0 0 rpy=0 0 1.57079632679, axis 0 0 0

File: robots/walkman/model.urdf (robot description, URDF)
Before this commit: robot bigman, 87 links, 86 joints
Links:
- added link LElb_fake, mass 0.0001
- added link LForearm_fake, mass 0.0001
- added link LShr_fake, mass 0.0001
- added link LShy_fake, mass 0.0001
- added link LWrMot2_fake, mass 0.0001
- added link LWrMot3_fake, mass 0.0001
- added link RElb_fake, mass 0.0001
- added link RForearm_fake, mass 0.0001
- added link RShr_fake, mass 0.0001
- added link RShy_fake, mass 0.0001
- added link RWrMot2_fake, mass 0.0001
- added link RWrMot3_fake, mass 0.0001
Joints:
- added joint j_LElb_fake: type fixed, parent LElb, child LElb_fake, origin xyz=0 0 0 rpy=-1.57079632679 0 0, axis 0 0 0
- added joint j_LForearm_fake: type fixed, parent LForearm, child LForearm_fake, origin xyz=0 0 0 rpy=-1.57079632679 0 0, axis 0 0 0
- added joint j_LShr_fake: type fixed, parent LShr, child LShr_fake, origin xyz=0 0 0 rpy=-1.57079632679 0 0, axis 0 0 0
- added joint j_LShy_fake: type fixed, parent LShy, child LShy_fake, origin xyz=0 0 0 rpy=-1.57079632679 0 0, axis 0 0 0
- added joint j_LWrMot2_fake: type fixed, parent LWrMot2, child LWrMot2_fake, origin xyz=0 0 0 rpy=-1.57079632679 0 0, axis 0 0 0
- added joint j_LWrMot3_fake: type fixed, parent LWrMot3, child LWrMot3_fake, origin xyz=0 0 0 rpy=-1.57079632679 0 0, axis 0 0 0
- added joint j_RElb_fake: type fixed, parent RElb, child RElb_fake, origin xyz=0 0 0 rpy=1.57079632679 0 0, axis 0 0 0
- added joint j_RForearm_fake: type fixed, parent RForearm, child RForearm_fake, origin xyz=0 0 0 rpy=1.57079632679 0 0, axis 0 0 0
- added joint j_RShr_fake: type fixed, parent RShr, child RShr_fake, origin xyz=0 0 0 rpy=1.57079632679 0 0, axis 0 0 0
- added joint j_RShy_fake: type fixed, parent RShy, child RShy_fake, origin xyz=0 0 0 rpy=1.57079632679 0 0, axis 0 0 0
- added joint j_RWrMot2_fake: type fixed, parent RWrMot2, child RWrMot2_fake, origin xyz=0 0 0 rpy=1.57079632679 0 0, axis 0 0 0
- added joint j_RWrMot3_fake: type fixed, parent RWrMot3, child RWrMot3_fake, origin xyz=0 0 0 rpy=1.57079632679 0 0, axis 0 0 0
