Commit message: update atlas urdf

File: robots/atlas/model.urdf (robot description, URDF)
Before this commit: robot atlas, 38 links, 37 joints
Links:
- added link l_hand_fake, mass 0.0001
- added link l_uarm_fake, mass 0.0001
- added link l_ufarm_fake, mass 0.0001
- added link r_hand_fake, mass 0.0001
- added link r_uarm_fake, mass 0.0001
- added link r_ufarm_fake, mass 0.0001
Joints:
- added joint j_l_hand_fake: type fixed, parent l_hand, child l_hand_fake, origin xyz=0 0 0 rpy=0 -1.57079632679 0, axis 0 0 0
- added joint j_l_uarm_fake: type fixed, parent l_uarm, child l_uarm_fake, origin xyz=0 0 0 rpy=0 -1.57079632679 0, axis 0 0 0
- added joint j_l_ufarm_fake: type fixed, parent l_ufarm, child l_ufarm_fake, origin xyz=0 0 0 rpy=0 -1.57079632679 0, axis 0 0 0
- added joint j_r_hand_fake: type fixed, parent r_hand, child r_hand_fake, origin xyz=0 0 0 rpy=0 -1.57079632679 0, axis 0 0 0
- added joint j_r_uarm_fake: type fixed, parent r_uarm, child r_uarm_fake, origin xyz=0 0 0 rpy=0 -1.57079632679 0, axis 0 0 0
- added joint j_r_ufarm_fake: type fixed, parent r_ufarm, child r_ufarm_fake, origin xyz=0 0 0 rpy=0 -1.57079632679 0, axis 0 0 0
